File: _restore_backup_2026-08-06T11-30-15-349/G-Love.kicad_sch (KiCad schematic)
At the start: 50 parts, among them U1 ATMEGA2561-16AU, U2 ATMega328P, Y1 16MHz, Y2 16MHz

Commit message: osekour
Connections:
- net VCC is gone; now on net +5V: C32.2, C33.1, J2.6, U2.18 (AVCC), U2.4 (VCC), U2.6 (VCC)
Changed lines of the file:
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@@
 	)
 	(junction
-		(at 167.64 44.45)
+		(at 43.18 176.53)
 		(diameter 0)
 		(color 0 0 0 0)
 	)
 	(junction
-		(at 43.18 176.53)
+		(at 167.64 44.45)
 		(diameter 0)
 		(color 0 0 0 0)
@@
 	)
 	(junction
+		(at 167.64 58.42)
+		(diameter 0)
+		(color 0 0 0 0)
+	)
+	(junction
 		(at 88.9 31.75)
 		(diameter 0)
@@
 	)
 	(junction
+		(at 97.79 31.75)
+		(diameter 0)
+		(color 0 0 0 0)
+	)
+	(junction
 		(at 196.85 30.48)
 		(diameter 0)
@@
 	(wire
 		(pts
+			(xy 167.64 58.42) (xy 167.64 44.45)
+		)
+		(stroke
+			(width 0)
+			(type default)
+		)
+	)
+	(wire
+		(pts
 			(xy 128.27 95.25) (xy 128.27 87.63)
 		)
@@
 	(wire
 		(pts
-			(xy 163.83 44.45) (xy 167.64 44.45)
-		)
-		(stroke
-			(width 0)
-			(type default)
-		)
-	)
-	(wire
-		(pts
 			(xy 213.36 90.17) (xy 252.73 90.17)
 		)
@@
 	(wire
 		(pts
+			(xy 100.33 31.75) (xy 97.79 31.75)
+		)
+		(stroke
+			(width 0)
+			(type default)
+		)
+	)
+	(wire
+		(pts
 			(xy 85.09 36.83) (xy 85.09 39.37)
 		)
@@
 	(wire
 		(pts
-			(xy 167.64 44.45) (xy 167.64 58.42)
-		)
-		(stroke
-			(width 0)
-			(type default)
-		)
-	)
-	(wire
-		(pts
 			(xy 46.99 40.64) (xy 49.53 40.64)
 		)
@@
 	(wire
 		(pts
+			(xy 167.64 58.42) (xy 167.64 59.69)
+		)
+		(stroke
+			(width 0)
+			(type default)
+		)
+	)
+	(wire
+		(pts
 			(xy 213.36 81.28) (xy 231.14 81.28)
 		)
@@
 		(in_pos_files yes)
 		(dnp no)
-		(property "Reference" "#PWR131"
+		(property "Reference" "#PWR0131"
 			(at 175.26 95.758 0)
 			(hide yes)
@@
 			(project "G-Love"
 				(path "/808bc5ea-49ac-4454-ba77-8b20d01ce159"
-					(reference "#PWR131")
+					(reference "#PWR0131")
 					(unit 1)
 				)
@@
 		(in_pos_files yes)
 		(dnp no)
-		(property "Reference" "#PWR124"
+		(property "Reference" "#PWR0124"
 			(at 97.79 22.098 0)
 			(hide yes)
@@
 			(project "G-Love"
 				(path "/808bc5ea-49ac-4454-ba77-8b20d01ce159"
-					(reference "#PWR124")
+					(reference "#PWR0124")
 					(unit 1)
 				)
@@
 		(in_pos_files yes)
 		(dnp no)
-		(property "Reference" "#PWR123"
+		(property "Reference" "#PWR0123"
 			(at 200.66 30.988 0)
 			(hide yes)
@@
 			)
 		)
-		(property "Value" "VCC"
+		(property "Value" "+5V"
 			(at 196.85 26.162 0)
 			(show_name no)
@@
 			(project "G-Love"
 				(path "/808bc5ea-49ac-4454-ba77-8b20d01ce159"
-					(reference "#PWR123")
+					(reference "#PWR0123")
 					(unit 1)
 				)
@@
 	(symbol
 		(lib_id "G-Love:GND")
-		(at 163.83 44.45 0)
+		(at 167.64 44.45 0)
 		(unit 1)
 		(body_style 1)
@@
 		(fields_autoplaced yes)
 		(property "Reference" "GND0143"
-			(at 163.83 48.006 0)
+			(at 167.64 48.006 0)
 			(hide yes)
 			(show_name no)
@@
 		)
 		(property "Value" "GND"
-			(at 163.83 48.006 0)
+			(at 167.64 48.006 0)
 			(hide yes)
 			(show_name no)
@@
 		)
 		(property "Footprint" ""
-			(at 163.83 44.45 0)
+			(at 167.64 44.45 0)
 			(hide yes)
 			(show_name no)
@@
 		)
 		(property "Datasheet" ""
-			(at 163.83 44.45 0)
+			(at 167.64 44.45 0)
 			(hide yes)
 			(show_name no)
@@
 		)
 		(property "Description" ""
-			(at 163.83 44.45 0)
+			(at 167.64 44.45 0)
 			(hide yes)
 			(show_name no)
@@
 		)
 		(property "Minimum quantity per command" ""
-			(at 163.83 44.45 0)
+			(at 167.64 44.45 0)
 			(hide yes)
 			(show_name no)
@@
 		(in_pos_files yes)
 		(dnp no)
-		(property "Reference" "#PWR141"
+		(property "Reference" "#PWR0141"
 			(at 148.59 62.738 0)
 			(hide yes)
@@
 			(project "G-Love"
 				(path "/808bc5ea-49ac-4454-ba77-8b20d01ce159"
-					(reference "#PWR141")
+					(reference "#PWR0141")
 					(unit 1)
 				)
@@
 		(dnp no)
 		(fields_autoplaced yes)
-		(property "Reference" "#PWR139"
+		(property "Reference" "#PWR0139"
 			(at 46.99 170.688 0)
 			(hide yes)
@@
 			(project "G-Love"
 				(path "/808bc5ea-49ac-4454-ba77-8b20d01ce159"
-					(reference "#PWR139")
+					(reference "#PWR0139")
 					(unit 1)
 				)
@@
 		(in_pos_files yes)
 		(dnp no)
-		(property "Reference" "#PWR142"
+		(property "Reference" "#PWR0142"
 			(at 256.54 110.998 0)
 			(hide yes)
@@
 			(project "G-Love"
 				(path "/808bc5ea-49ac-4454-ba77-8b20d01ce159"
-					(reference "#PWR142")
+					(reference "#PWR0142")
 					(unit 1)
 				)
