File: _restore_backup_2026-08-06T11-30-15-349/hallCaptor.kicad_sch (KiCad schematic)
At the start: 1 part

Commit message: osekour
Parts:
- removed J_3: (no value), MyGlove:PinHeader_1x04_Pas2.54mm, symbol G-Love:Conn_POGO_4
- added U6: Hall Sensor A3144, MyGlove:Hall_Sensor_A3144, symbol G-Love:A3144
Connections:
- net GND: now also U6.2 (GND)
- new net +3.3V: U6.1 (VCC)
- new net HallGPIO_Clasp: U6.3 (Output)
