File: _restore_backup_2026-08-06T11-30-15-349/outputs.kicad_sch (KiCad schematic)
At the start: 22 parts, among them U9 TUSB321

Commit message: osekour
Parts:
- J_5: symbol G-Love:J_USB_RECEPTACLE_PASSIVE -> G-Love:J_USB_RECEPTACLE
Connections:
- net VCC is gone; now on net +5V: C23.2, U9.12 (VDD)
Changed lines of the file:
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@@
 	)
 	(symbol
-		(lib_id "G-Love:J_USB_RECEPTACLE_PASSIVE")
+		(lib_name "J_USB_RECEPTACLE_1")
+		(lib_id "G-Love:J_USB_RECEPTACLE")
 		(at 66.04 151.13 0)
 		(unit 1)
@@
 		(dnp no)
 		(fields_autoplaced yes)
-		(property "Reference" "#PWR1"
+		(property "Reference" "#PWR01"
 			(at 143.51 27.178 0)
 			(hide yes)
@@
 			)
 		)
-		(property "Value" "VCC"
+		(property "Value" "+5V"
 			(at 139.7 21.59 0)
 			(show_name no)
@@
 			(project "G-Love"
 				(path "/808bc5ea-49ac-4454-ba77-8b20d01ce159/0d387f9d-76d6-4b6a-aded-93bcda75ef5a"
-					(reference "#PWR1")
+					(reference "#PWR01")
 					(unit 1)
 				)
@@
 		(dnp no)
 		(fields_autoplaced yes)
-		(property "Reference" "#PWR15"
+		(property "Reference" "#PWR015"
 			(at 118.11 53.848 0)
 			(hide yes)
@@
 			(project "G-Love"
 				(path "/808bc5ea-49ac-4454-ba77-8b20d01ce159/0d387f9d-76d6-4b6a-aded-93bcda75ef5a"
-					(reference "#PWR15")
+					(reference "#PWR015")
 					(unit 1)
 				)
