File: touchscreen.kicad_sch (KiCad schematic)
At the start: 7 parts, among them U3 TXS0108EPWR, U7 GC9A01_TFT, U8 CST816D

Commit message: up
Parts:
- removed C34, C35: 100nF, MyGlove:Capacitor_0603, symbol G-Love:C
- removed D107: RED, MyGlove:LED, symbol G-Love:LED_Indicator
- removed R39: 1k, MyGlove:Resistor_0603, symbol G-Love:R
- added C52, C53: 100nF, MyGlove:Capacitor_0603, symbol G-Love:C
- U3: renamed from U8; footprint MyGlove:PinHeader_1x04_Pas2.54mm -> MyGlove:PinHeader_1x04_P2.54mm_Vertical_CST816D
- U4: renamed from U7; footprint MyGlove:PinHeader_1x08_Pas2.54mm -> MyGlove:PinHeader_1x08_P2.54mm_Vertical
- renumbered U3 to U5
Connections:
- net +3.3V: now also C53.1
- net GND: now also C52.1, C53.2
- net VCC: now also C52.2

Commit message: Fini
Parts:
- removed C52, C53: 100nF, MyGlove:Capacitor_0603, symbol G-Love:C
- added D3: RED, MyGlove:LED, symbol G-Love:LED_Indicator
- added R19: 1k, MyGlove:Resistor_0603, symbol G-Love:R
- U3: footprint MyGlove:PinHeader_1x04_P2.54mm_Vertical_CST816D -> MyGlove:PinHeader_1x04_Pas2.54mm
- U4: footprint MyGlove:PinHeader_1x08_P2.54mm_Vertical -> MyGlove:PinHeader_1x08_Pas2.54mm
Connections:
- net +3.3V: now also R19.1
- net GND: now also D3.2 (K)
- new net: D3.1 (A), R19.2

Commit message: reste routage mais peu
Parts:
- U3: footprint MyGlove:PinHeader_1x04_Pas2.54mm -> MyGlove:PinHeader_1x04_P2.54mm_Vertical
- U4: footprint MyGlove:PinHeader_1x08_Pas2.54mm -> MyGlove:PinHeader_1x08_P2.54mm_Vertical
Changed lines of the file:
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@@
 			)
 		)
-		(property "Footprint" "MyGlove:PinHeader_1x04_Pas2.54mm"
+		(property "Footprint" "MyGlove:PinHeader_1x04_P2.54mm_Vertical"
 			(at 91.44 119.38 0)
 			(hide yes)
@@
 			)
 		)
-		(property "Footprint" "MyGlove:PinHeader_1x08_Pas2.54mm"
+		(property "Footprint" "MyGlove:PinHeader_1x08_P2.54mm_Vertical"
 			(at 93.98 64.77 0)
 			(hide yes)

Commit message: Regles de design
Parts:
- D3: footprint MyGlove:LED -> MyGlove:D_0603_1608Metric_Pad1.05x0.95mm_HandSolder
- U3: footprint MyGlove:PinHeader_1x04_P2.54mm_Vertical -> MyGlove:PinHeader_1x04_Pas2.54mm_cst816d
Changed lines of the file:
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@@
 			)
 		)
-		(property "Footprint" "MyGlove:PinHeader_1x04_P2.54mm_Vertical"
+		(property "Footprint" "MyGlove:PinHeader_1x04_Pas2.54mm_cst816d"
 			(at 91.44 119.38 0)
 			(hide yes)
@@
 			)
 		)
-		(property "Footprint" "MyGlove:LED"
+		(property "Footprint" "MyGlove:D_0603_1608Metric_Pad1.05x0.95mm_HandSolder"
 			(at 104.14 40.64 0)
 			(hide yes)

Commit message: Debut potable
Parts:
- removed D3: RED, MyGlove:D_0603_1608Metric_Pad1.05x0.95mm_HandSolder, symbol G-Love:LED_Indicator
- removed R19: 1k, MyGlove:Resistor_0603, symbol G-Love:R

Commit message: Passe ERC
Parts:
- added C52, C53: 100nF, MyGlove:Capacitor_0603, symbol G-Love:C
- U3: footprint MyGlove:PinHeader_1x04_Pas2.54mm_cst816d -> MyGlove:PinHeader_1x04_P2.54mm_Vertical_CST816D
Connections:
- net +3.3V: now also C53.1
- net GND: now also C52.1, C53.2
- net VCC: now also C52.2
