File: G-Love.kicad_pcb (KiCad board)
At the start: 2 copper layers, 130.4 x 73.5 mm, 154 parts, among them J4 XLR5_Ground, U14 TPS2113APWR, U18 MAX485E, Y1 16MHz, Y2 16MHz

Commit message: up
Parts:
- moved D102 3.89 mm to (55.3, 61.1), turned to 90 degrees
- moved D101 3.74 mm to (49.9, 48.1), turned to -90 degrees
- moved R19 2.60 mm to (114.1, 74.9)
- moved C52 1.91 mm to (87.0, 51.4)
- moved R22 1.60 mm to (87.1, 53.1)
- moved R18 1.56 mm to (85.9, 95.3)
- moved R17 1.46 mm to (85.9, 93.8)
- moved R20 1.20 mm to (114.2, 77.4)
- moved C16 0.81 mm to (125.8, 76.0)
- moved C18 0.78 mm to (123.6, 73.8)
- moved C17 0.78 mm to (124.7, 74.9)
- moved C23 0.11 mm to (52.3, 66.7), turned to 180 degrees
- turned C20 to 180 degrees
Routing:
- net VCC: track 460.2 -> 479.4 mm, vias 7 -> 9
- net Net-(B0505S-1W2-0V): track 102.2 -> 98.1 mm
- net Net-(D101-K): track 7.46 -> 4.88 mm
- net GND: track 64.8 -> 62.3 mm
- net /Data/power I/O/2561_UART_TX: track 28.5 -> 26.1 mm
- net /FingerTip Modules/FingerTip_I2C_SDA: track 68.6 -> 66.4 mm, vias 2 -> 3
- net /Hand_Captors/I2C_IMU_SDA: track 10.3 -> 8.27 mm
- net /Hand_Captors/I2C_IMU_SDK: track 17.2 -> 15.8 mm
- net /Hand_Captors/ADC_X_Output: track 16.8 -> 15.4 mm
- net /FingerTip Modules/FingerTip_I2C_SCL: track 61.2 -> 60.1 mm
- net +3.3V: track 191.7 -> 191.1 mm

Commit message: fix: route under instead of between resistor and capacitor
Routing:
- net VBUS: track 117.5 -> 118.1 mm

Commit message: up
Routing:
- net /Data/power I/O/Data/UD-: track 29.2 -> 32.2 mm
- net Net-(U10-X0): track 14.9 -> 16.7 mm
- net +3.3V: track 191.1 -> 192.7 mm
- net /Hand_Captors/Flex_Sensor0/FlexADC: track 16.3 -> 17.7 mm
- net /MCU_328_RESET: track 64.4 -> 63.3 mm
- net VBUS: track 118.1 -> 118.8 mm
- net /Hand_Captors/ADC_Mux_Select_C: track 20.0 -> 19.4 mm
- net /Hand_Captors/FSR_Thumb/TouchADC: track 26.5 -> 27.1 mm

Commit message: fix routing and carrefour
Routing:
- net /Data/power I/O/Data/UD-: track 32.2 -> 30.0 mm

Commit message: up
Routing:
- net VCC: track 479.5 -> 514.1 mm, vias 9 -> 12
- net GND: track 62.3 -> 71.0 mm, vias 30 -> 34
- net VBUS: track 118.8 -> 124.4 mm
- net /MCU_2561_RESET: track 55.5 -> 54.5 mm
- net Net-(J_1-CC1): track 37.7 -> 38.4 mm
