File: SK9822_O.kicad_sch (KiCad schematic)
At the start: 5 parts

Commit message: reste routage mais peu
Parts:
- D24: footprint MyGlove:PinHeader_1x02_Pas2.54mm_ -> MyGlove:PinHeader_1x02_P2.54mm_Vertical
Changed lines of the file:
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@@
 			)
 		)
-		(property "Footprint" "MyGlove:PinHeader_1x02_Pas2.54mm_"
+		(property "Footprint" "MyGlove:PinHeader_1x02_P2.54mm_Vertical"
 			(at 41.91 36.83 0)
 			(hide yes)

Commit message: up
Parts:
- renumbered D24 to D23, D25 to D24, D26 to D25, D27 to D26, D28 to D27
Changed lines of the file:
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@@
 		(dnp no)
 		(fields_autoplaced yes)
-		(property "Reference" "D25"
+		(property "Reference" "D24"
 			(at 65.6433 22.86 0)
 			(show_name no)
@@
 			(project "G-Love"
 				(path "/808bc5ea-49ac-4454-ba77-8b20d01ce159/80069e6d-e99d-4fb8-a6cc-8c9cf1821a0c/508c8d26-610d-4395-9434-749869aaa3fc/cb06373c-fd44-4fb3-af88-6af9d82061bd"
-					(reference "D25")
+					(reference "D24")
 					(unit 1)
 				)
@@
 		(dnp no)
 		(fields_autoplaced yes)
-		(property "Reference" "D24"
+		(property "Reference" "D23"
 			(at 44.0533 22.86 0)
 			(show_name no)
@@
 			(project "G-Love"
 				(path "/808bc5ea-49ac-4454-ba77-8b20d01ce159/80069e6d-e99d-4fb8-a6cc-8c9cf1821a0c/508c8d26-610d-4395-9434-749869aaa3fc/cb06373c-fd44-4fb3-af88-6af9d82061bd"
-					(reference "D24")
+					(reference "D23")
 					(unit 1)
 				)
@@
 		(dnp no)
 		(fields_autoplaced yes)
-		(property "Reference" "D27"
+		(property "Reference" "D26"
 			(at 108.8233 22.86 0)
 			(show_name no)
@@
 			(project "G-Love"
 				(path "/808bc5ea-49ac-4454-ba77-8b20d01ce159/80069e6d-e99d-4fb8-a6cc-8c9cf1821a0c/508c8d26-610d-4395-9434-749869aaa3fc/cb06373c-fd44-4fb3-af88-6af9d82061bd"
-					(reference "D27")
+					(reference "D26")
 					(unit 1)
 				)
@@
 		(dnp no)
 		(fields_autoplaced yes)
-		(property "Reference" "D26"
+		(property "Reference" "D25"
 			(at 87.2333 22.86 0)
 			(show_name no)
@@
 			(project "G-Love"
 				(path "/808bc5ea-49ac-4454-ba77-8b20d01ce159/80069e6d-e99d-4fb8-a6cc-8c9cf1821a0c/508c8d26-610d-4395-9434-749869aaa3fc/cb06373c-fd44-4fb3-af88-6af9d82061bd"
-					(reference "D26")
+					(reference "D25")
 					(unit 1)
 				)
@@
 		(dnp no)
 		(fields_autoplaced yes)
-		(property "Reference" "D28"
+		(property "Reference" "D27"
 			(at 130.4133 22.86 0)
 			(show_name no)
@@
 			(project "G-Love"
 				(path "/808bc5ea-49ac-4454-ba77-8b20d01ce159/80069e6d-e99d-4fb8-a6cc-8c9cf1821a0c/508c8d26-610d-4395-9434-749869aaa3fc/cb06373c-fd44-4fb3-af88-6af9d82061bd"
-					(reference "D28")
+					(reference "D27")
 					(unit 1)
 				)
