File: _restore_backup_2026-08-12T12-55-47-787/FSR.kicad_sch (KiCad schematic)
At the start: 3 parts

Commit message: Fini
Parts:
- FSR1: renamed from FSR_1; footprint MyGlove:PinHeader_1x02_Pas2.54mm_ -> MyGlove:PinHeader_1x02_P2.54mm_Vertical
- renumbered C13 to C14
Changed lines of the file:
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@@
 		(in_pos_files yes)
 		(dnp no)
-		(property "Reference" "C13"
+		(property "Reference" "C14"
 			(at 32.004 47.244 0)
 			(show_name no)
@@
 			(project "G-Love"
 				(path "/808bc5ea-49ac-4454-ba77-8b20d01ce159/c9027db4-6968-4e40-a138-b60eacbff4db/15052d3f-5b94-4226-97e2-3e9ab10fafda"
-					(reference "C13")
+					(reference "C14")
 					(unit 1)
 				)
 				(path "/808bc5ea-49ac-4454-ba77-8b20d01ce159/c9027db4-6968-4e40-a138-b60eacbff4db/32c3dc22-6eac-49d0-b512-767615f82205"
-					(reference "C14")
+					(reference "C15")
 					(unit 1)
 				)
 				(path "/808bc5ea-49ac-4454-ba77-8b20d01ce159/c9027db4-6968-4e40-a138-b60eacbff4db/3f48e459-1dc8-4eb9-8adc-befbe01eab22"
+					(reference "C17")
+					(unit 1)
+				)
+				(path "/808bc5ea-49ac-4454-ba77-8b20d01ce159/c9027db4-6968-4e40-a138-b60eacbff4db/5442b494-eff8-4ddd-bc03-bcc1bea75842"
 					(reference "C16")
 					(unit 1)
 				)
-				(path "/808bc5ea-49ac-4454-ba77-8b20d01ce159/c9027db4-6968-4e40-a138-b60eacbff4db/5442b494-eff8-4ddd-bc03-bcc1bea75842"
-					(reference "C15")
-					(unit 1)
-				)
 				(path "/808bc5ea-49ac-4454-ba77-8b20d01ce159/c9027db4-6968-4e40-a138-b60eacbff4db/f906f610-f118-4325-955e-6566f843376d"
-					(reference "C17")
+					(reference "C18")
 					(unit 1)
 				)
@@
 		(in_pos_files yes)
 		(dnp no)
-		(property "Reference" "FSR_1"
+		(property "Reference" "FSR1"
 			(at 20.828 30.48 0)
 			(show_name no)
@@
 			)
 		)
-		(property "Footprint" "MyGlove:PinHeader_1x02_Pas2.54mm_"
+		(property "Footprint" "MyGlove:PinHeader_1x02_P2.54mm_Vertical"
 			(at 24.13 30.48 0)
 			(hide yes)
@@
 			(project "G-Love"
 				(path "/808bc5ea-49ac-4454-ba77-8b20d01ce159/c9027db4-6968-4e40-a138-b60eacbff4db/15052d3f-5b94-4226-97e2-3e9ab10fafda"
-					(reference "FSR_1")
+					(reference "FSR1")
 					(unit 1)
 				)
 				(path "/808bc5ea-49ac-4454-ba77-8b20d01ce159/c9027db4-6968-4e40-a138-b60eacbff4db/32c3dc22-6eac-49d0-b512-767615f82205"
-					(reference "FSR_2")
+					(reference "FSR2")
 					(unit 1)
 				)
 				(path "/808bc5ea-49ac-4454-ba77-8b20d01ce159/c9027db4-6968-4e40-a138-b60eacbff4db/3f48e459-1dc8-4eb9-8adc-befbe01eab22"
-					(reference "FSR_4")
+					(reference "FSR4")
 					(unit 1)
 				)
 				(path "/808bc5ea-49ac-4454-ba77-8b20d01ce159/c9027db4-6968-4e40-a138-b60eacbff4db/5442b494-eff8-4ddd-bc03-bcc1bea75842"
-					(reference "FSR_3")
+					(reference "FSR3")
 					(unit 1)
 				)
 				(path "/808bc5ea-49ac-4454-ba77-8b20d01ce159/c9027db4-6968-4e40-a138-b60eacbff4db/f906f610-f118-4325-955e-6566f843376d"
-					(reference "FSR_5")
+					(reference "FSR5")
 					(unit 1)
 				)
@@
 		(dnp no)
 		(fields_autoplaced yes)
-		(property "Reference" "GND011"
+		(property "Reference" "GND012"
 			(at 24.13 61.976 0)
 			(hide yes)
@@
 			(project "G-Love"
 				(path "/808bc5ea-49ac-4454-ba77-8b20d01ce159/c9027db4-6968-4e40-a138-b60eacbff4db/15052d3f-5b94-4226-97e2-3e9ab10fafda"
-					(reference "GND011")
+					(reference "GND012")
 					(unit 1)
 				)
 				(path "/808bc5ea-49ac-4454-ba77-8b20d01ce159/c9027db4-6968-4e40-a138-b60eacbff4db/32c3dc22-6eac-49d0-b512-767615f82205"
-					(reference "GND012")
+					(reference "GND013")
 					(unit 1)
 				)
 				(path "/808bc5ea-49ac-4454-ba77-8b20d01ce159/c9027db4-6968-4e40-a138-b60eacbff4db/3f48e459-1dc8-4eb9-8adc-befbe01eab22"
+					(reference "GND015")
+					(unit 1)
+				)
+				(path "/808bc5ea-49ac-4454-ba77-8b20d01ce159/c9027db4-6968-4e40-a138-b60eacbff4db/5442b494-eff8-4ddd-bc03-bcc1bea75842"
 					(reference "GND014")
 					(unit 1)
 				)
-				(path "/808bc5ea-49ac-4454-ba77-8b20d01ce159/c9027db4-6968-4e40-a138-b60eacbff4db/5442b494-eff8-4ddd-bc03-bcc1bea75842"
-					(reference "GND013")
-					(unit 1)
-				)
 				(path "/808bc5ea-49ac-4454-ba77-8b20d01ce159/c9027db4-6968-4e40-a138-b60eacbff4db/f906f610-f118-4325-955e-6566f843376d"
-					(reference "GND015")
-					(unit 1)
-				)
+					(reference "GND016")
+					(unit 1)
+				)
