File: _restore_backup_2026-08-12T12-55-47-787/G-Love.kicad_pcb (KiCad board)
At the start: 2 copper layers, 70.3 x 95.2 mm, 152 parts, among them J3 XLR5_Ground, U1 ATMEGA2561-16AU, U10 74HC4052, U11 TUSB321, U12 TPS2113APWR, U13 AMS1117, U14 6N137, U15 MAX485E, U2 ATMega328P, U3 CST816D, U4 GC9A01_TFT, U5 TXS0108EPWR, U6 ICM-42688-P_I2C, U7 TXS0104E, U8 Hall Sensor A3144, U9 74HC4052, Y1 16MHz, Y2 16MHz

Commit message: Fini
Parts:
- removed REF** (x12): NPTH_Drill_Hole, MyGlove:NPTH_Drill_Hole
