File: _restore_backup_2026-08-12T12-55-47-787/captors.kicad_sch (KiCad schematic)
At the start: 1 part

Commit message: Fini
Parts:
- added C32: 100nF, MyGlove:Capacitor_0603, symbol G-Love:C
Connections:
- net ADC_Mux_Inhibit is gone; now on net GND: CD1.13 (INHIBIT)
- net ADC_Mux_Select_B: now also CD1.14 (C); no longer CD1.11 (B)
- net ADC_Mux_Select_C: now also CD1.11 (B); no longer CD1.14 (C)
- net GND: now also C32.1
- net VCC: now also C32.2
