File: _restore_backup_2026-08-12T12-55-47-787/fingertip.kicad_sch (KiCad schematic)
At the start: 1 part

Commit message: Fini
Parts:
- J_3: footprint MyGlove:PinHeader_1x04_Pas2.54mm -> MyGlove:PinHeader_1x04_P2.54mm_Vertical
Changed lines of the file:
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@@
 		(dnp no)
 		(fields_autoplaced yes)
-		(property "Reference" "GND0159"
+		(property "Reference" "GND0161"
 			(at 55.88 83.566 0)
 			(hide yes)
@@
 			(project "G-Love"
 				(path "/808bc5ea-49ac-4454-ba77-8b20d01ce159/8701d982-557e-4c73-bfaa-5f02d2e6c25d"
-					(reference "GND0159")
+					(reference "GND0161")
 					(unit 1)
 				)
@@
 			)
 		)
-		(property "Footprint" "MyGlove:PinHeader_1x04_Pas2.54mm"
+		(property "Footprint" "MyGlove:PinHeader_1x04_P2.54mm_Vertical"
 			(at 72.39 72.39 0)
 			(hide yes)
