File: _restore_backup_2026-08-12T12-55-47-787/power.kicad_sch (KiCad schematic)
At the start: 14 parts, among them U12 TPS2113APWR, U13 AMS1117

Commit message: Fini
Parts:
- renumbered C36 to C38, C37 to C39, C38 to C40, C39 to C41, C40 to C42, C41 to C43, C42 to C44, C43 to C45, R34 to R33, R35 to R34, R36 to R35, R37 to R36
Changed lines of the file:
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@@
 		(exclude_from_sim no)
 		(in_bom yes)
-		(on_board yes)
+		(on_board no)
 		(in_pos_files yes)
 		(dnp no)
-		(property "Reference" "C39"
+		(property "Reference" "C41"
 			(at 54.61 63.246 0)
 			(show_name no)
@@
 			(project "G-Love"
 				(path "/808bc5ea-49ac-4454-ba77-8b20d01ce159/0d387f9d-76d6-4b6a-aded-93bcda75ef5a/0a598795-0604-41b3-948f-4efe200200e3"
-					(reference "C39")
+					(reference "C41")
 					(unit 1)
 				)
@@
 		(dnp no)
 		(fields_autoplaced yes)
-		(property "Reference" "GND0157"
+		(property "Reference" "GND0159"
 			(at 91.44 175.006 0)
 			(hide yes)
@@
 			(project "G-Love"
 				(path "/808bc5ea-49ac-4454-ba77-8b20d01ce159/0d387f9d-76d6-4b6a-aded-93bcda75ef5a/0a598795-0604-41b3-948f-4efe200200e3"
-					(reference "GND0157")
+					(reference "GND0159")
 					(unit 1)
 				)
@@
 		(in_pos_files yes)
 		(dnp no)
-		(property "Reference" "C42"
+		(property "Reference" "C44"
 			(at 143.51 155.194 0)
 			(show_name no)
@@
 			(project "G-Love"
 				(path "/808bc5ea-49ac-4454-ba77-8b20d01ce159/0d387f9d-76d6-4b6a-aded-93bcda75ef5a/0a598795-0604-41b3-948f-4efe200200e3"
-					(reference "C42")
+					(reference "C44")
 					(unit 1)
 				)
@@
 		(dnp no)
 		(fields_autoplaced yes)
-		(property "Reference" "GND0153"
+		(property "Reference" "GND0155"
 			(at 50.8 171.196 0)
 			(hide yes)
@@
 			(project "G-Love"
 				(path "/808bc5ea-49ac-4454-ba77-8b20d01ce159/0d387f9d-76d6-4b6a-aded-93bcda75ef5a/0a598795-0604-41b3-948f-4efe200200e3"
-					(reference "GND0153")
+					(reference "GND0155")
 					(unit 1)
 				)
@@
 		(dnp no)
 		(fields_autoplaced yes)
-		(property "Reference" "GND0158"
+		(property "Reference" "GND0160"
 			(at 130.81 166.116 0)
 			(hide yes)
@@
 			(project "G-Love"
 				(path "/808bc5ea-49ac-4454-ba77-8b20d01ce159/0d387f9d-76d6-4b6a-aded-93bcda75ef5a/0a598795-0604-41b3-948f-4efe200200e3"
-					(reference "GND0158")
+					(reference "GND0160")
 					(unit 1)
 				)
@@
 		(dnp no)
 		(fields_autoplaced yes)
-		(property "Reference" "GND0152"
+		(property "Reference" "GND0154"
 			(at 41.91 157.226 0)
 			(hide yes)
@@
 			(project "G-Love"
 				(path "/808bc5ea-49ac-4454-ba77-8b20d01ce159/0d387f9d-76d6-4b6a-aded-93bcda75ef5a/0a598795-0604-41b3-948f-4efe200200e3"
-					(reference "GND0152")
+					(reference "GND0154")
 					(unit 1)
 				)
@@
 		(in_pos_files yes)
 		(dnp no)
-		(property "Reference" "C38"
+		(property "Reference" "C40"
 			(at 51.562 163.068 0)
 			(show_name no)
@@
 			(project "G-Love"
 				(path "/808bc5ea-49ac-4454-ba77-8b20d01ce159/0d387f9d-76d6-4b6a-aded-93bcda75ef5a/0a598795-0604-41b3-948f-4efe200200e3"
-					(reference "C38")
+					(reference "C40")
 					(unit 1)
 				)
@@
 		(dnp no)
 		(fields_autoplaced yes)
-		(property "Reference" "C40"
+		(property "Reference" "C42"
 			(at 93.98 158.3181 0)
 			(show_name no)
@@
 			(project "G-Love"
 				(path "/808bc5ea-49ac-4454-ba77-8b20d01ce159/0d387f9d-76d6-4b6a-aded-93bcda75ef5a/0a598795-0604-41b3-948f-4efe200200e3"
-					(reference "C40")
+					(reference "C42")
 					(unit 1)
 				)
@@
 		(exclude_from_sim no)
 		(in_bom yes)
-		(on_board yes)
+		(on_board no)
 		(in_pos_files yes)
 		(dnp no)
-		(property "Reference" "R35"
+		(property "Reference" "R34"
 			(at 67.31 64.7699 90)
 			(show_name no)
@@
 			(project "G-Love"
 				(path "/808bc5ea-49ac-4454-ba77-8b20d01ce159/0d387f9d-76d6-4b6a-aded-93bcda75ef5a/0a598795-0604-41b3-948f-4efe200200e3"
-					(reference "R35")
+					(reference "R34")
 					(unit 1)
 				)
@@
 		(dnp no)
 		(fields_autoplaced yes)
-		(property "Reference" "GND0154"
+		(property "Reference" "GND0156"
 			(at 53.34 73.406 0)
 			(hide yes)
@@
 			(project "G-Love"
 				(path "/808bc5ea-49ac-4454-ba77-8b20d01ce159/0d387f9d-76d6-4b6a-aded-93bcda75ef5a/0a598795-0604-41b3-948f-4efe200200e3"
-					(reference "GND0154")
+					(reference "GND0156")
 					(unit 1)
 				)
@@
 		(in_pos_files yes)
 		(dnp no)
-		(property "Reference" "R34"
+		(property "Reference" "R33"
 			(at 47.498 152.654 0)
 			(show_name no)
@@
 			(project "G-Love"
 				(path "/808bc5ea-49ac-4454-ba77-8b20d01ce159/0d387f9d-76d6-4b6a-aded-93bcda75ef5a/0a598795-0604-41b3-948f-4efe200200e3"
-					(reference "R34")
+					(reference "R33")
 					(unit 1)
 				)
@@
 		(in_pos_files yes)
 		(dnp no)
-		(property "Reference" "C41"
+		(property "Reference" "C43"
 			(at 113.03 156.21 0)
 			(show_name no)
@@
 			(project "G-Love"
 				(path "/808bc5ea-49ac-4454-ba77-8b20d01ce159/0d387f9d-76d6-4b6a-aded-93bcda75ef5a/0a598795-0604-41b3-948f-4efe200200e3"
-					(reference "C41")
+					(reference "C43")
 					(unit 1)
 				)
@@
 		(exclude_from_sim no)
 		(in_bom yes)
-		(on_board yes)
+		(on_board no)
 		(in_pos_files yes)
 		(dnp no)
-		(property "Reference" "C36"
+		(property "Reference" "C38"
 			(at 41.91 63.246 0)
 			(show_name no)
@@
 			(project "G-Love"
 				(path "/808bc5ea-49ac-4454-ba77-8b20d01ce159/0d387f9d-76d6-4b6a-aded-93bcda75ef5a/0a598795-0604-41b3-948f-4efe200200e3"
-					(reference "C36")
+					(reference "C38")
 					(unit 1)
 				)
@@
 		(dnp no)
 		(fields_autoplaced yes)
-		(property "Reference" "GND0151"
+		(property "Reference" "GND0153"
 			(at 40.64 73.406 0)
 			(hide yes)
@@
 			(project "G-Love"
 				(path "/808bc5ea-49ac-4454-ba77-8b20d01ce159/0d387f9d-76d6-4b6a-aded-93bcda75ef5a/0a598795-0604-41b3-948f-4efe200200e3"
-					(reference "GND0151")
+					(reference "GND0153")
 					(unit 1)
 				)
@@
 		(in_pos_files yes)
 		(dnp no)
-		(property "Reference" "R36"
+		(property "Reference" "R35"
 			(at 86.868 145.796 90)
 			(show_name no)
@@
 			(project "G-Love"
 				(path "/808bc5ea-49ac-4454-ba77-8b20d01ce159/0d387f9d-76d6-4b6a-aded-93bcda75ef5a/0a598795-0604-41b3-948f-4efe200200e3"
-					(reference "R36")
+					(reference "R35")
 					(unit 1)
 				)
@@
 		(in_pos_files yes)
 		(dnp no)
-		(property "Reference" "C37"
+		(property "Reference" "C39"
 			(at 45.212 163.068 0)
 			(show_name no)
@@
 			(project "G-Love"
 				(path "/808bc5ea-49ac-4454-ba77-8b20d01ce159/0d387f9d-76d6-4b6a-aded-93bcda75ef5a/0a598795-0604-41b3-948f-4efe200200e3"
-					(reference "C37")
+					(reference "C39")
 					(unit 1)
 				)
@@
 		(in_pos_files yes)
 		(dnp no)
-		(property "Reference" "R37"
+		(property "Reference" "R36"
 			(at 90.932 145.796 90)
 			(show_name no)
@@
 			(project "G-Love"
 				(path "/808bc5ea-49ac-4454-ba77-8b20d01ce159/0d387f9d-76d6-4b6a-aded-93bcda75ef5a/0a598795-0604-41b3-948f-4efe200200e3"
-					(reference "R37")
+					(reference "R36")
 					(unit 1)
 				)
@@
 		(dnp no)
 		(fields_autoplaced yes)
-		(property "Reference" "GND0156"
+		(property "Reference" "GND0158"
 			(at 90.17 152.146 0)
 			(hide yes)
@@
 			(project "G-Love"
 				(path "/808bc5ea-49ac-4454-ba77-8b20d01ce159/0d387f9d-76d6-4b6a-aded-93bcda75ef5a/0a598795-0604-41b3-948f-4efe200200e3"
-					(reference "GND0156")
+					(reference "GND0158")
 					(unit 1)
 				)
@@
 		(in_pos_files yes)
 		(dnp no)
-		(property "Reference" "C43"
+		(property "Reference" "C45"
 			(at 151.13 155.194 0)
 			(show_name no)
@@
 			(project "G-Love"
 				(path "/808bc5ea-49ac-4454-ba77-8b20d01ce159/0d387f9d-76d6-4b6a-aded-93bcda75ef5a/0a598795-0604-41b3-948f-4efe200200e3"
-					(reference "C43")
+					(reference "C45")
 					(unit 1)
 				)
@@
 		(dnp no)
 		(fields_autoplaced yes)
-		(property "Reference" "GND0155"
+		(property "Reference" "GND0157"
 			(at 66.04 74.676 0)
 			(hide yes)
@@
 			(project "G-Love"
 				(path "/808bc5ea-49ac-4454-ba77-8b20d01ce159/0d387f9d-76d6-4b6a-aded-93bcda75ef5a/0a598795-0604-41b3-948f-4efe200200e3"
-					(reference "GND0155")
+					(reference "GND0157")
 					(unit 1)
 				)
