File: Kicad/V1/fingertip.kicad_sch (KiCad schematic)
At the start: 1 part

Commit message: ERC Check
Parts:
- J_3: footprint MyGlove:PinHeader_1x04_Pas2.54mm -> MyGlove:PinHeader_1x04_P2.54mm_Vertical
Changed lines of the file:
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@@
 			)
 		)
-		(property "Footprint" "MyGlove:PinHeader_1x04_Pas2.54mm"
+		(property "Footprint" "MyGlove:PinHeader_1x04_P2.54mm_Vertical"
 			(at 72.39 72.39 0)
 			(hide yes)
