File: Kicad/V1/ATMega2561.kicad_sch (KiCad schematic)
At the start: 32 parts, among them U16 ATMEGA2561-16AU, Y3 16MHz

Commit message: ERC almost done, footprint to assign
Parts:
- U5: renamed from U16; footprint MyGlove:ATMega2561 -> G-Love:ATMEGA2561-16AU; PACKAGE (none) -> QFP-64
- renumbered C50 to C19, C51 to C20, C1 to C21, C2 to C22, C53 to C23, C52 to C24, C54 to C25, J1 to J4, R1 to R17, SW_1 to SW_2, TP20 to TP1, TP28 to TP10, TP29 to TP11, TP30 to TP12, TP31 to TP13, TP32 to TP14, TP33 to TP15, TP34 to TP16, TP35 to TP17, TP36 to TP18, TP19 to TP2, TP21 to TP3, TP22 to TP4, TP23 to TP5, TP24 to TP6, TP25 to TP7, TP26 to TP8, TP27 to TP9, Y3 to Y2, flow19 to flow5, flow20 to flow6
Connections:
- net MCU_328_RESET: no longer names the net of U5.35 (PC0_(A8))
- no-connect marks 22 -> 23

Commit message: ERC Check
Parts:
- J4: footprint MyGlove:PinHeader_1x06_Pas2.54mm -> MyGlove:PinHeader_1x06_P2.54mm_Vertical
- U5: footprint G-Love:ATMEGA2561-16AU -> MyGlove:ATMega2561
Changed lines of the file:
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@@
 			)
 		)
-		(property "Footprint" "MyGlove:PinHeader_1x06_Pas2.54mm"
+		(property "Footprint" "MyGlove:PinHeader_1x06_P2.54mm_Vertical"
 			(at 34.29 181.61 0)
 			(hide yes)
@@
 			)
 		)
-		(property "Footprint" "G-Love:ATMEGA2561-16AU"
+		(property "Footprint" "MyGlove:ATMega2561"
 			(at 157.48 157.226 0)
 			(hide yes)

Commit message: add gnd to 2560 quatrz
Connections:
- net GND: now also C19.2, C20.1
Changed lines of the file:
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@@
+		(color 0 0 0 0)
+	)
+	(junction
+		(at 101.6 53.34)
+		(diameter 0)
 		(color 0 0 0 0)
 	)
@@
 	(wire
 		(pts
+			(xy 101.6 53.34) (xy 101.6 59.69)
+		)
+		(stroke
+			(width 0)
+			(type default)
+		)
+	)
+	(wire
+		(pts
 			(xy 152.4 43.18) (xy 156.21 43.18)
 		)
@@
 	(wire
 		(pts
-			(xy 101.6 46.99) (xy 101.6 59.69)
+			(xy 101.6 46.99) (xy 101.6 53.34)
 		)
 		(stroke
@@
 	(wire
 		(pts
+			(xy 99.06 53.34) (xy 101.6 53.34)
+		)
+		(stroke
+			(width 0)
+			(type default)
+		)
+	)
+	(wire
+		(pts
 			(xy 167.64 127) (xy 191.77 127)
 		)
@@
 	(wire
 		(pts
-			(xy 104.14 53.34) (xy 105.41 53.34)
-		)
-		(stroke
-			(width 0)
-			(type default)
-		)
-	)
-	(wire
-		(pts
 			(xy 82.55 93.98) (xy 121.92 93.98)
 		)
@@
 		(pts
 			(xy 167.64 134.62) (xy 191.77 134.62)
+		)
+		(stroke
+			(width 0)
+			(type default)
+		)
+	)
+	(wire
+		(pts
+			(xy 101.6 53.34) (xy 105.41 53.34)
 		)
 		(stroke
@@
 	(symbol
 		(lib_id "G-Love:GND")
-		(at 104.14 53.34 0)
+		(at 99.06 53.34 0)
+		(mirror y)
 		(unit 1)
 		(body_style 1)
@@
 		(dnp no)
 		(property "Reference" "#GND02"
-			(at 104.14 56.896 0)
+			(at 99.06 56.896 0)
 			(hide yes)
 			(show_name no)
@@
 		)
 		(property "Value" "GND"
-			(at 102.108 56.896 90)
+			(at 101.092 56.896 90)
 			(hide yes)
 			(show_name no)
@@
 		)
 		(property "Footprint" ""
-			(at 104.14 53.34 0)
+			(at 99.06 53.34 0)
 			(hide yes)
 			(show_name no)
@@
 		)
 		(property "Datasheet" ""
-			(at 104.14 53.34 0)
+			(at 99.06 53.34 0)
 			(hide yes)
 			(show_name no)
@@
 		)
 		(property "Description" ""
-			(at 104.14 53.34 0)
-			(hide yes)
-			(show_name no)
+			(at 99.06 53.34 0)
+			(hide yes)
+			(show_name no)

Commit message: correction 328p et ajout d'un capa
Parts:
- renumbered C19 to C20, C20 to C21, C21 to C22, C22 to C23, C23 to C24, C24 to C25, C25 to C26
Changed lines of the file:
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@@
 		(in_pos_files yes)
 		(dnp no)
-		(property "Reference" "C25"
+		(property "Reference" "C26"
 			(at 157.48 45.212 90)
 			(show_name no)
@@
 			(project "G-Love"
 				(path "/808bc5ea-49ac-4454-ba77-8b20d01ce159/8591a7a3-fa5a-416e-b459-40b6a5958f2a"
-					(reference "C25")
+					(reference "C26")
 					(unit 1)
 				)
@@
 		(in_pos_files yes)
 		(dnp no)
-		(property "Reference" "C20"
+		(property "Reference" "C21"
 			(at 105.156 57.912 90)
 			(show_name no)
@@
 			(project "G-Love"
 				(path "/808bc5ea-49ac-4454-ba77-8b20d01ce159/8591a7a3-fa5a-416e-b459-40b6a5958f2a"
-					(reference "C20")
+					(reference "C21")
 					(unit 1)
 				)
@@
 		(in_pos_files yes)
 		(dnp no)
-		(property "Reference" "C19"
+		(property "Reference" "C20"
 			(at 105.156 42.672 90)
 			(show_name no)
@@
 			(project "G-Love"
 				(path "/808bc5ea-49ac-4454-ba77-8b20d01ce159/8591a7a3-fa5a-416e-b459-40b6a5958f2a"
-					(reference "C19")
+					(reference "C20")
 					(unit 1)
 				)
@@
 		(in_pos_files yes)
 		(dnp no)
-		(property "Reference" "C24"
+		(property "Reference" "C25"
 			(at 155.702 37.846 90)
 			(show_name no)
@@
 			(project "G-Love"
 				(path "/808bc5ea-49ac-4454-ba77-8b20d01ce159/8591a7a3-fa5a-416e-b459-40b6a5958f2a"
-					(reference "C24")
+					(reference "C25")
 					(unit 1)
 				)
@@
 		(in_pos_files yes)
 		(dnp no)
-		(property "Reference" "C21"
+		(property "Reference" "C22"
 			(at 113.284 184.15 90)
 			(show_name no)
@@
 			(project "G-Love"
 				(path "/808bc5ea-49ac-4454-ba77-8b20d01ce159/8591a7a3-fa5a-416e-b459-40b6a5958f2a"
-					(reference "C21")
+					(reference "C22")
 					(unit 1)
 				)
@@
 		(in_pos_files yes)
 		(dnp no)
-		(property "Reference" "C23"
+		(property "Reference" "C24"
 			(at 156.718 32.004 90)
 			(show_name no)
@@
 			(project "G-Love"
 				(path "/808bc5ea-49ac-4454-ba77-8b20d01ce159/8591a7a3-fa5a-416e-b459-40b6a5958f2a"
-					(reference "C23")
+					(reference "C24")
 					(unit 1)
 				)
@@
 		(in_pos_files yes)
 		(dnp no)
-		(property "Reference" "C22"
+		(property "Reference" "C23"
 			(at 130.048 185.674 0)
 			(show_name no)
@@
 			(project "G-Love"
 				(path "/808bc5ea-49ac-4454-ba77-8b20d01ce159/8591a7a3-fa5a-416e-b459-40b6a5958f2a"
-					(reference "C22")
+					(reference "C23")
 					(unit 1)
 				)
