File: Kicad/V1/ATmega328P_sch.kicad_sch (KiCad schematic)
At the start: 14 parts, among them J4 SPI_LED, U2 ATMega328P, Y2 16MHz

Commit message: ERC almost done, footprint to assign
Parts:
- renumbered C8 to C1, C9 to C2, C10 to C4, C11 to C5, C12 to C6, J2 to J1, J4 to J2, R4 to R5, SW_2 to SW_1, U2 to U1, Y2 to Y1
Connections:
- net MCU_328_RESET is gone; now on net MCU_328P_RESET: U1.29 (~{RESET}/PCINT14/PC6)
- net 328P_I2C_IMU_SCK renamed 328P_I2C_IMU_SCL

Commit message: ERC Check
Parts:
- J1: footprint MyGlove:PinHeader_1x06_Pas2.54mm -> MyGlove:PinHeader_1x06_P2.54mm_Vertical
- J2: footprint (none) -> MyGlove:PinHeader_1x02_P2.54mm_Vertical
Changed lines of the file:
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@@
 			)
 		)
-		(property "Footprint" ""
+		(property "Footprint" "MyGlove:PinHeader_1x02_P2.54mm_Vertical"
 			(at 226.06 60.96 0)
 			(hide yes)
@@
 			)
 		)
-		(property "Footprint" "MyGlove:PinHeader_1x06_Pas2.54mm"
+		(property "Footprint" "MyGlove:PinHeader_1x06_P2.54mm_Vertical"
 			(at 24.13 182.88 0)
 			(hide yes)

Commit message: correction 328p et ajout d'un capa
Parts:
- added C2: 100nF, MyGlove:Capacitor_0603, symbol G-Love:C
- renumbered C2 to C3, C3 to C4, C4 to C5, C5 to C6, C6 to C7
Connections:
- net GND: now also C2.1
- net VCC: now also C2.2
Other:
- moved on the sheet: C3, C5
