File: Kicad/V1/IMU.kicad_sch (KiCad schematic)
At the start: 5 parts, among them U6 ICM-42688-P_I2C, U7 TXS0104E

Commit message: ERC almost done, footprint to assign
Parts:
- renumbered C24 to C7, C25 to C8, C26 to C9, U6 to U2, U7 to U3
Connections:
- net IMU_I2C_SDK renamed IMU_I2C_SCL
Changed lines of the file:
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@@
 		)
 	)
-	(hierarchical_label "IMU_I2C_SDK"
+	(hierarchical_label "IMU_I2C_SCL"
 		(shape input)
 		(at 151.13 62.23 0)
@@
 		(in_pos_files yes)
 		(dnp no)
-		(property "Reference" "U6"
+		(property "Reference" "U2"
 			(at 54.102 78.486 0)
 			(show_name no)
@@
 			(project "G-Love"
 				(path "/808bc5ea-49ac-4454-ba77-8b20d01ce159/7de4e8e6-4751-4acb-b71f-e492a47c8332/f73c6c7b-472d-4c5d-b434-31d2ac317fba"
-					(reference "U6")
+					(reference "U2")
 					(unit 1)
 				)
@@
 		(in_pos_files yes)
 		(dnp no)
-		(property "Reference" "GND029"
+		(property "Reference" "GND011"
 			(at 76.2 55.626 0)
 			(hide yes)
@@
 			(project "G-Love"
 				(path "/808bc5ea-49ac-4454-ba77-8b20d01ce159/7de4e8e6-4751-4acb-b71f-e492a47c8332/f73c6c7b-472d-4c5d-b434-31d2ac317fba"
-					(reference "GND029")
+					(reference "GND011")
+					(unit 1)
+				)
+			)
+		)
+	)
+	(symbol
+		(lib_id "G-Love:VCC")
+		(at 140.97 48.26 0)
+		(unit 1)
+		(body_style 1)
+		(exclude_from_sim no)
+		(in_bom no)
+		(on_board no)
+		(in_pos_files yes)
+		(dnp no)
+		(fields_autoplaced yes)
+		(property "Reference" "#PWR011"
+			(at 144.78 50.038 0)
+			(hide yes)
+			(show_name no)
+			(do_not_autoplace no)
+			(effects
+				(font
+					(size 1.27 1.27)
+				)
+			)
+		)
+		(property "Value" "VCC"
+			(at 140.97 44.45 0)
+			(show_name no)
+			(do_not_autoplace no)
+			(effects
+				(font
+					(size 1.27 1.27)
+				)
+			)
+		)
+		(property "Footprint" ""
+			(at 140.97 48.26 0)
+			(hide yes)
+			(show_name no)
+			(do_not_autoplace no)
+			(effects
+				(font
+					(size 1.27 1.27)
+				)
+			)
+		)
+		(property "Datasheet" ""
+			(at 140.97 48.26 0)
+			(hide yes)
+			(show_name no)
+			(do_not_autoplace no)
+			(effects
+				(font
+					(size 1.27 1.27)
+				)
+			)
+		)
+		(property "Description" ""
+			(at 140.97 48.26 0)
+			(hide yes)
+			(show_name no)
+			(do_not_autoplace no)
+			(effects
+				(font
+					(size 1.27 1.27)
+				)
+			)
+		)
+		(pin "1"
+		)
+		(instances
+			(project "G-Love"
+				(path "/808bc5ea-49ac-4454-ba77-8b20d01ce159/7de4e8e6-4751-4acb-b71f-e492a47c8332/f73c6c7b-472d-4c5d-b434-31d2ac317fba"
+					(reference "#PWR011")
 					(unit 1)
 				)
@@
 		(in_pos_files yes)
 		(dnp no)
-		(property "Reference" "C25"
+		(property "Reference" "C8"
 			(at 72.39 40.64 90)
 			(show_name no)
@@
 			(project "G-Love"
 				(path "/808bc5ea-49ac-4454-ba77-8b20d01ce159/7de4e8e6-4751-4acb-b71f-e492a47c8332/f73c6c7b-472d-4c5d-b434-31d2ac317fba"
-					(reference "C25")
+					(reference "C8")
 					(unit 1)
 				)
@@
 		(in_pos_files yes)
 		(dnp no)
-		(property "Reference" "GND027"
+		(property "Reference" "GND09"
 			(at 73.66 84.836 0)
 			(hide yes)
@@
 			(project "G-Love"
 				(path "/808bc5ea-49ac-4454-ba77-8b20d01ce159/7de4e8e6-4751-4acb-b71f-e492a47c8332/f73c6c7b-472d-4c5d-b434-31d2ac317fba"
-					(reference "GND027")
+					(reference "GND09")
 					(unit 1)
 				)
@@
 		(in_pos_files yes)
 		(dnp no)
-		(property "Reference" "GND026"
+		(property "Reference" "GND08"
 			(at 53.34 51.816 0)
 			(hide yes)
@@
 			(project "G-Love"
 				(path "/808bc5ea-49ac-4454-ba77-8b20d01ce159/7de4e8e6-4751-4acb-b71f-e492a47c8332/f73c6c7b-472d-4c5d-b434-31d2ac317fba"
-					(reference "GND026")
+					(reference "GND08")
 					(unit 1)
 				)
@@
 		(in_pos_files yes)
 		(dnp no)
-		(property "Reference" "#PWR024"
+		(property "Reference" "#PWR08"
 			(at 66.04 41.148 0)
 			(hide yes)
@@
 			(project "G-Love"
 				(path "/808bc5ea-49ac-4454-ba77-8b20d01ce159/7de4e8e6-4751-4acb-b71f-e492a47c8332/f73c6c7b-472d-4c5d-b434-31d2ac317fba"
-					(reference "#PWR024")
+					(reference "#PWR08")
 					(unit 1)
 				)
@@
 		(in_pos_files yes)
 		(dnp no)
-		(property "Reference" "GND030"
+		(property "Reference" "GND012"
 			(at 135.89 82.296 0)
 			(hide yes)
@@
 			(project "G-Love"
 				(path "/808bc5ea-49ac-4454-ba77-8b20d01ce159/7de4e8e6-4751-4acb-b71f-e492a47c8332/f73c6c7b-472d-4c5d-b434-31d2ac317fba"
-					(reference "GND030")
+					(reference "GND012")
 					(unit 1)
 				)
@@
 		(in_pos_files yes)
 		(dnp no)
-		(property "Reference" "C26"
+		(property "Reference" "C9"
 			(at 71.628 46.99 90)
 			(show_name no)
@@
 			(project "G-Love"
 				(path "/808bc5ea-49ac-4454-ba77-8b20d01ce159/7de4e8e6-4751-4acb-b71f-e492a47c8332/f73c6c7b-472d-4c5d-b434-31d2ac317fba"
-					(reference "C26")
+					(reference "C9")
 					(unit 1)
 				)
@@
 		(in_pos_files yes)
 		(dnp no)
-		(property "Reference" "GND028"
+		(property "Reference" "GND010"
 			(at 76.2 49.276 0)
 			(hide yes)
@@
 			(project "G-Love"
 				(path "/808bc5ea-49ac-4454-ba77-8b20d01ce159/7de4e8e6-4751-4acb-b71f-e492a47c8332/f73c6c7b-472d-4c5d-b434-31d2ac317fba"
-					(reference "GND028")
+					(reference "GND010")
 					(unit 1)
 				)
@@
 		(in_pos_files yes)
 		(dnp no)
-		(property "Reference" "C24"
+		(property "Reference" "C7"
 			(at 57.658 42.418 90)
 			(show_name no)
@@
 			(project "G-Love"
 				(path "/808bc5ea-49ac-4454-ba77-8b20d01ce159/7de4e8e6-4751-4acb-b71f-e492a47c8332/f73c6c7b-472d-4c5d-b434-31d2ac317fba"
-					(reference "C24")
-					(unit 1)
-				)
-			)
-		)
-	)
-	(symbol
-		(lib_id "G-Love:VCC")
-		(at 140.97 48.26 0)
-		(unit 1)
-		(body_style 1)
-		(exclude_from_sim no)
-		(in_bom no)
-		(on_board no)
-		(in_pos_files yes)
-		(dnp no)
-		(property "Reference" "#PWR027"
-			(at 144.78 50.038 0)
-			(hide yes)
-			(show_name no)
-			(do_not_autoplace no)
-			(effects
-				(font
-					(size 1.27 1.27)
-				)
-			)
-		)
-		(property "Value" "VCC"
-			(at 143.256 46.482 0)
-			(show_name no)
-			(do_not_autoplace no)
-			(effects
-				(font
-					(size 1.27 1.27)
-				)
-			)
-		)
-		(property "Footprint" ""
-			(at 140.97 48.26 0)
-			(hide yes)
-			(show_name no)
-			(do_not_autoplace no)
-			(effects
-				(font
-					(size 1.27 1.27)
-				)
-			)
-		)
-		(property "Datasheet" ""
-			(at 140.97 48.26 0)
-			(hide yes)
-			(show_name no)
-			(do_not_autoplace no)
-			(effects
-				(font
-					(size 1.27 1.27)
-				)
-			)
-		)
-		(property "Description" ""
-			(at 140.97 48.26 0)
-			(hide yes)
-			(show_name no)
-			(do_not_autoplace no)
-			(effects
-				(font
-					(size 1.27 1.27)
-				)
-			)
-		)
-		(pin "1"
-		)
-		(instances
-			(project "G-Love"
-				(path "/808bc5ea-49ac-4454-ba77-8b20d01ce159/7de4e8e6-4751-4acb-b71f-e492a47c8332/f73c6c7b-472d-4c5d-b434-31d2ac317fba"
-					(reference "#PWR027")
+					(reference "C7")
 					(unit 1)
 				)
@@
 		(in_pos_files yes)
 		(dnp no)
-		(property "Reference" "#PWR025"
+		(property "Reference" "#PWR09"
 			(at 71.12 41.148 0)
 			(hide yes)
@@
 			(project "G-Love"
 				(path "/808bc5ea-49ac-4454-ba77-8b20d01ce159/7de4e8e6-4751-4acb-b71f-e492a47c8332/f73c6c7b-472d-4c5d-b434-31d2ac317fba"
-					(reference "#PWR025")
+					(reference "#PWR09")
 					(unit 1)
 				)
@@
 		(in_pos_files yes)
 		(dnp no)
-		(property "Reference" "U7"
+		(property "Reference" "U3"
 			(at 144.018 80.772 0)
 			(show_name no)
@@
 			(project "G-Love"
 				(path "/808bc5ea-49ac-4454-ba77-8b20d01ce159/7de4e8e6-4751-4acb-b71f-e492a47c8332/f73c6c7b-472d-4c5d-b434-31d2ac317fba"
-					(reference "U7")
+					(reference "U3")
 					(unit 1)
 				)
@@
 		(in_pos_files yes)
 		(dnp no)
-		(property "Reference" "#PWR026"
+		(property "Reference" "#PWR010"
 			(at 139.7 50.038 0)
 			(hide yes)
@@
 			(project "G-Love"
 				(path "/808bc5ea-49ac-4454-ba77-8b20d01ce159/7de4e8e6-4751-4acb-b71f-e492a47c8332/f73c6c7b-472d-4c5d-b434-31d2ac317fba"
-					(reference "#PWR026")
+					(reference "#PWR010")
 					(unit 1)
 				)

Commit message: correction 328p et ajout d'un capa
Parts:
- renumbered C9 to C10, C7 to C8, C8 to C9
Changed lines of the file:
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@@
 		(in_pos_files yes)
 		(dnp no)
-		(property "Reference" "C8"
+		(property "Reference" "C9"
 			(at 72.39 40.64 90)
 			(show_name no)
@@
 			(project "G-Love"
 				(path "/808bc5ea-49ac-4454-ba77-8b20d01ce159/7de4e8e6-4751-4acb-b71f-e492a47c8332/f73c6c7b-472d-4c5d-b434-31d2ac317fba"
-					(reference "C8")
+					(reference "C9")
 					(unit 1)
 				)
@@
 		(in_pos_files yes)
 		(dnp no)
-		(property "Reference" "C9"
+		(property "Reference" "C10"
 			(at 71.628 46.99 90)
 			(show_name no)
@@
 			(project "G-Love"
 				(path "/808bc5ea-49ac-4454-ba77-8b20d01ce159/7de4e8e6-4751-4acb-b71f-e492a47c8332/f73c6c7b-472d-4c5d-b434-31d2ac317fba"
-					(reference "C9")
+					(reference "C10")
 					(unit 1)
 				)
@@
 		(in_pos_files yes)
 		(dnp no)
-		(property "Reference" "C7"
+		(property "Reference" "C8"
 			(at 57.658 42.418 90)
 			(show_name no)
@@
 			(project "G-Love"
 				(path "/808bc5ea-49ac-4454-ba77-8b20d01ce159/7de4e8e6-4751-4acb-b71f-e492a47c8332/f73c6c7b-472d-4c5d-b434-31d2ac317fba"
-					(reference "C7")
+					(reference "C8")
 					(unit 1)
 				)
