File: Kicad/V1/switch.kicad_sch (KiCad schematic)
At the start: 25 parts, among them U10 74HC4052, U9 74HC4052

Commit message: ERC almost done, footprint to assign
Parts:
- renumbered C27 to C33, C28 to C34, C29 to C35, C30 to C36, D104 to D5, D105 to D6, R20 to R30, R21 to R31, R22 to R32, R23 to R33, U9 to U7, U10 to U8, flow6 to flow10, flow7 to flow11, flow8 to flow12, flow9 to flow13, flow10 to flow14, flow11 to flow15, flow12 to flow16, flow13 to flow17, flow14 to flow18, flow15 to flow19, flow16 to flow20, flow5 to flow9

Commit message: correction 328p et ajout d'un capa
Parts:
- renumbered C33 to C34, C34 to C35, C35 to C36, C36 to C37
Changed lines of the file:
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@@
 		(in_pos_files yes)
 		(dnp no)
-		(property "Reference" "C35"
+		(property "Reference" "C36"
 			(at 77.47 85.344 0)
 			(show_name no)
@@
 			(project "G-Love"
 				(path "/808bc5ea-49ac-4454-ba77-8b20d01ce159/0d387f9d-76d6-4b6a-aded-93bcda75ef5a/4989b515-8901-47ca-ab95-4d280b30f712"
-					(reference "C35")
+					(reference "C36")
 					(unit 1)
 				)
@@
 		(in_pos_files yes)
 		(dnp no)
-		(property "Reference" "C34"
+		(property "Reference" "C35"
 			(at 71.12 129.54 90)
 			(show_name no)
@@
 			(project "G-Love"
 				(path "/808bc5ea-49ac-4454-ba77-8b20d01ce159/0d387f9d-76d6-4b6a-aded-93bcda75ef5a/4989b515-8901-47ca-ab95-4d280b30f712"
-					(reference "C34")
+					(reference "C35")
 					(unit 1)
 				)
@@
 		(in_pos_files yes)
 		(dnp no)
-		(property "Reference" "C36"
+		(property "Reference" "C37"
 			(at 185.42 88.646 0)
 			(show_name no)
@@
 			(project "G-Love"
 				(path "/808bc5ea-49ac-4454-ba77-8b20d01ce159/0d387f9d-76d6-4b6a-aded-93bcda75ef5a/4989b515-8901-47ca-ab95-4d280b30f712"
-					(reference "C36")
+					(reference "C37")
 					(unit 1)
 				)
@@
 		(in_pos_files yes)
 		(dnp no)
-		(property "Reference" "C33"
+		(property "Reference" "C34"
 			(at 62.23 123.444 90)
 			(show_name no)
@@
 			(project "G-Love"
 				(path "/808bc5ea-49ac-4454-ba77-8b20d01ce159/0d387f9d-76d6-4b6a-aded-93bcda75ef5a/4989b515-8901-47ca-ab95-4d280b30f712"
-					(reference "C33")
+					(reference "C34")
 					(unit 1)
 				)
