File: Kicad/V1/_restore_backup_2026-09-07T15-01-36-097/G-Love.kicad_pcb (KiCad board)
At the start: 2 copper layers, 36 x 36 mm, 154 parts, among them J5 XLR5_Ground, U1 ATMega328P, U10 6N137, U11 MAX485E, U12 TPS2113APWR, U13 AMS1117, U2 ICM-42688-P_I2C, U3 TXS0104E, U4 Hall Sensor A3144, U5 ATMEGA2561-16AU, U6 TUSB321, U7 74HC4052, U8 74HC4052, U9 B0505S-1W1, Y1 16MHz, Y2 16MHz

Commit message: correction schema elec + ajout connecteur FPC
Parts:
- added J1: ~, MyGlove:PinHeader_1x06_P2.54mm_Vertical, F.Cu at (133.2, 104.0)
- added J2: SPI_LED, MyGlove:PinHeader_1x02_P2.54mm_Vertical, F.Cu at (146.3, 110.1)
- moved R7 54.2 mm to (141.9, 113.9), turned to 0 degrees
- moved R6 53.1 mm to (141.9, 111.4), turned to 0 degrees
- moved C7 3.05 mm to (211.6, 106.7), turned to 0 degrees
- moved C6 0.70 mm to (206.1, 108.2)
