File: Kicad/V1/_restore_backup_2026-09-07T15-01-36-097/captors.kicad_sch (KiCad schematic)
At the start: 1 part

Commit message: correction schema elec + ajout connecteur FPC
Other:
- removed sheet hand_captors
Changed lines of the file:
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@@
-	)
-	(sheet
-		(at 234.95 60.96)
-		(size 31.75 46.99)
-		(exclude_from_sim no)
-		(in_bom yes)
-		(on_board yes)
-		(dnp no)
-		(fields_autoplaced yes)
-		(stroke
-			(width 0.1524)
-			(type solid)
-		)
-		(fill
-			(color 0 0 0 0)
-		)
-		(property "Sheetname" "hand_captors"
-			(at 234.95 60.2484 0)
-			(show_name no)
-			(do_not_autoplace no)
-			(effects
-				(font
-					(size 1.27 1.27)
-				)
-				(justify left bottom)
-			)
-		)
-		(property "Sheetfile" "hand_captors.kicad_sch"
-			(at 234.95 108.5346 0)
-			(show_name no)
-			(do_not_autoplace no)
-			(effects
-				(font
-					(size 1.27 1.27)
-				)
-				(justify left top)
-			)
-		)
-		(instances
-			(project "G-Love"
-				(path "/808bc5ea-49ac-4454-ba77-8b20d01ce159/7de4e8e6-4751-4acb-b71f-e492a47c8332"
-					(page "24")
-				)
-			)
-		)
 	)
 	(sheet
