File: Kicad/V2/Schematic/hand_captors.kicad_sch (KiCad schematic)
At the start: 21 parts

Commit message: Split power and data
Parts:
- renumbered C40 to C35, C41 to C36, C42 to C37, C43 to C38, C44 to C39, C45 to C40, C46 to C41, C47 to C42, C48 to C43, C49 to C44, R33 to R26, R34 to R27, R35 to R28, R36 to R29, R37 to R30, R38 to R31, R39 to R32, R40 to R33, R41 to R34, R42 to R35, R43 to R36
