File: Kicad/V2/Schematic/captors.kicad_sch (KiCad schematic)
At the start: 7 parts, among them U2 TXS0104E

Commit message: Alimentation finalisée & blindage connecteur FPC
Connections:
- net +3.3V: now also J2.8 (3.3V); no longer J2.4 (3.3V)
- net GND: now also J2.11 (GND), J2.18 (GND), J2.24 (GND), J2.3 (GND), J2.4 (GND), J2.7 (GND); no longer J2.20 (GND)
- net I2C_IMU_SCL: now also U2.12 (B2); no longer U2.13 (B1)
- net I2C_IMU_SDA: now also U2.13 (B1); no longer U2.12 (B2)
- net VCC: no longer J2.1 (VCC), J2.2 (VCCL), J2.3 (VCCL)
- net hand_captors/FLEX_INDEX_IN: now also J2.16 (FLEX_INDEX); no longer J2.11 (INDEX_FLEX)
- net hand_captors/FLEX_LITTLE_IN: now also J2.23 (FLEX_LITTLE); no longer J2.19 (FLEX_LITTLE)
- net hand_captors/FLEX_MIDDLE_IN: now also J2.19 (FLEX_MIDDLE); no longer J2.15 (FLEX_MIDDLE)
- net hand_captors/FLEX_RING_IN: now also J2.21 (FLEX_RING); no longer J2.17 (FLEX_RING)
- net hand_captors/FLEX_THUMB_IN: now also J2.14 (FLEX_THUMB); no longer J2.9 (THUMB_FLEX)
- net hand_captors/FORCE_INDEX_IN: now also J2.15 (FSR_INDEX); no longer J2.10 (INDEX_FORCE)
- net hand_captors/FORCE_LITTLE_IN: now also J2.22 (FORCE_LITTLE); no longer J2.18 (FORCE_LITTLE)
- net hand_captors/FORCE_MIDDLE_IN: now also J2.17 (FSR_MIDDLE); no longer J2.14 (FORCE_MIDDLE)
- net hand_captors/FORCE_RING_IN: now also J2.20 (FORCE_RING); no longer J2.16 (FORCE_RING)
- net hand_captors/FORCE_THUMB_IN: now also J2.13 (FSR_THUMB); no longer J2.8 (THUMB_FORCE)
- net hand_captors/HALL_IN: now also J2.12 (SW_HALL); no longer J2.7 (HALL)
- net at R11.1, U2.2 (A1): now also J2.9 (SDA); no longer J2.13 (IMU_SCL)
- net at R10.1, U2.3 (A2): now also J2.10 (SCL); no longer J2.12 (IMU_SDA)
- new net VCCL: J2.1 (VCCL), J2.2 (VCCL)

Commit message: New footprints : Ferrite bead, poly fuse, TVS diode. To do: FPC connector footprint
Parts:
- added D3, D4, D5, D6: (no value), MyGlove:TVS_DIODE, symbol G-Love:TVS_ARRAY
- C8, C9: footprint (none) -> MyGlove:Capacitor_0603
- R12: renamed from R10; footprint (none) -> MyGlove:Resistor_0603
- R13: renamed from R11; footprint (none) -> MyGlove:Resistor_0603
Connections:
- net +3.3V: now also R12.2, R13.2
- net GND: now also D3.3, D4.3, D5.3, D6.3
- net LED_MOSI: now also D3.2
- net LED_SCK: now also D3.1
- net VCC: no longer R12.2, R13.2
- net hand_captors/FLEX_INDEX_IN: now also D6.5
- net hand_captors/FLEX_LITTLE_IN: now also D4.4
- net hand_captors/FLEX_MIDDLE_IN: now also D6.2
- net hand_captors/FLEX_RING_IN: now also D4.1
- net hand_captors/FLEX_THUMB_IN: now also D5.4
- net hand_captors/FORCE_INDEX_IN: now also D5.5
- net hand_captors/FORCE_LITTLE_IN: now also D4.2
- net hand_captors/FORCE_MIDDLE_IN: now also D6.4
- net hand_captors/FORCE_RING_IN: now also D6.1
- net hand_captors/FORCE_THUMB_IN: now also D5.2
- net hand_captors/HALL_IN: now also D5.1
- net at J2.9 (SDA), R13.1, U2.2 (A1): now also D3.4
- net at J2.10 (SCL), R12.1, U2.3 (A2): now also D3.5
- no-connect marks 10 -> 11

Commit message: final V2.0
Parts:
- removed D4, D5, D6: (no value), MyGlove:TVS_DIODE, symbol G-Love:TVS_ARRAY
- J2: footprint (none) -> G-Love:FPC_CONNECTOR_24
Connections:
- no-connect marks 11 -> 10
