File: Kicad/V2/Schematic/switch.kicad_sch (KiCad schematic)
At the start: 31 parts, among them J4 Conn_USB_Receptacle, U4 CH340K, U5 74HC4052

Commit message: New footprints : Ferrite bead, poly fuse, TVS diode. To do: FPC connector footprint
Parts:
- R20: renamed from R19; footprint (none) -> MyGlove:Resistor_0603
- R21: renamed from R20; footprint (none) -> MyGlove:Resistor_0603
- R22: renamed from R21; footprint (none) -> MyGlove:Resistor_0603
- renumbered C17 to C15, C18 to C16, C19 to C17, C20 to C18, D6 to D10, D4 to D8, D5 to D9, J5 to J3, J4 to J_2, R17 to R18, R18 to R19, R22 to R23, R23 to R24, R24 to R25, R25 to R26, U5 to U4, U4 to U_1
Connections:
- net GND: now also J3.1 (GND), J3.4 (GND); no longer J3.3
- net at U4.5 (Y1): now also J3.2 (Tx); no longer J3.1
- net at U4.14 (X1): now also J3.3 (Rx); no longer J3.2

Commit message: final V2.0
Parts:
- J3: footprint (none) -> G-Love:JST 4 Pin
Connections:
- net VCC: no longer C16.2, U_1.7 (VCC)
- net PC_DETECT: no longer names the net of R20.2
- net PC_DETECT: now also C16.2, U_1.7 (VCC)
Changed lines of the file:
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@@
 	(wire
 		(pts
-			(xy 77.47 88.9) (xy 119.38 88.9)
+			(xy 77.47 88.9) (xy 129.54 88.9)
 		)
 		(stroke
@@
 	(wire
 		(pts
-			(xy 129.54 101.6) (xy 129.54 110.49)
-		)
-		(stroke
-			(width 0)
-			(type default)
-		)
-	)
-	(hierarchical_label "PC_DETECT"
-		(shape output)
-		(at 119.38 88.9 0)
-		(effects
-			(font
-				(size 1.27 1.27)
-			)
-			(justify left)
+			(xy 129.54 88.9) (xy 129.54 110.49)
+		)
+		(stroke
+			(width 0)
+			(type default)
 		)
 	)
@@
 			)
 		)
-		(property "Footprint" ""
+		(property "Footprint" "G-Love:JST 4 Pin"
 			(at 166.37 74.93 0)
 			(hide yes)
@@
 					(unit 1)
 				)
-			)
-		)
-	)
-	(symbol
-		(lib_id "G-Love:VCC")
-		(at 129.54 100.33 0)
-		(unit 1)
-		(body_style 1)
-		(exclude_from_sim no)
-		(in_bom no)
-		(on_board no)
-		(in_pos_files yes)
-		(dnp no)
-		(fields_autoplaced yes)
-		(property "Reference" "#PWR017"
-			(at 133.35 102.108 0)
-			(hide yes)
-			(show_name no)
-			(do_not_autoplace no)
-			(effects
-				(font
-					(size 1.27 1.27)
-				)
-			)
-		)
-		(property "Value" "VCC"
-			(at 129.54 96.52 0)
-			(show_name no)
-			(do_not_autoplace no)
-			(effects
-				(font
-					(size 1.27 1.27)
-				)
-			)
-		)
-		(property "Footprint" ""
-			(at 129.54 100.33 0)
-			(hide yes)
-			(show_name no)
-			(do_not_autoplace no)
-			(effects
-				(font
-					(size 1.27 1.27)
-				)
-			)
-		)
-		(property "Datasheet" ""
-			(at 129.54 100.33 0)
-			(hide yes)
-			(show_name no)
-			(do_not_autoplace no)
-			(effects
-				(font
-					(size 1.27 1.27)
-				)
-			)
-		)
-		(property "Description" ""
-			(at 129.54 100.33 0)
-			(hide yes)
-			(show_name no)
-			(do_not_autoplace no)
-			(effects
-				(font
-					(size 1.27 1.27)
-				)
-			)
-		)
-		(pin "1"
-		)
-		(instances
-			(project "G-Love"
-				(path "/808bc5ea-49ac-4454-ba77-8b20d01ce159/bda75adb-ac63-42a7-b1e7-5ba80bc60aa7"
-					(reference "#PWR017")
-					(unit 1)
-				)
