File: Kicad/V2/Schematic/_restore_backup_2026-09-09T17-30-15-719/hand_captors.kicad_sch (KiCad schematic)
At the start: 21 parts

Commit message: finition schematic de reference
Parts:
- renumbered C34 to C35, C35 to C36, C36 to C37, C37 to C38, C38 to C39, C39 to C40, C40 to C41, C41 to C42, C42 to C43, C43 to C44, R30 to R26, R31 to R27, R32 to R28, R33 to R29, R34 to R30, R35 to R31, R36 to R32, R37 to R33, R38 to R34, R39 to R35, R40 to R36
