File: Kicad/V2/Schematic/_restore_backup_2026-09-09T17-30-15-719/switch.kicad_sch (KiCad schematic)
At the start: 31 parts, among them J4 Conn_USB_Receptacle, U4 CH340K, U5 74HC4052

Commit message: finition schematic de reference
Parts:
- removed J4: Conn_USB_Receptacle, MyGlove:USB_C_Receptacle_GCT_USB4105-xx-A_16P_TopMnt_Horizontal, symbol G-Love:J_USB_RECEPTACLE_PASSIVE
- added J8: Conn_USB_Receptacle, MyGlove:USB_C_Receptacle_GCT_USB4105-xx-A_16P_TopMnt_Horizontal, symbol G-Love:J_USB_RECEPTACLE
- renumbered C17 to C25, C18 to C45, C19 to C46, C20 to C47, D4 to D7, D5 to D8, D6 to D9, J5 to J9, R17 to R40, R18 to R41, R19 to R42, R20 to R43, R21 to R44, R22 to R45, R23 to R46, R24 to R47, R25 to R48, U4 to U10, U5 to U11, flow3 to flow21, flow4 to flow22, flow5 to flow23, flow6 to flow24, flow7 to flow25, flow8 to flow26, flow9 to flow27, flow10 to flow28, flow11 to flow29, flow12 to flow30, flow13 to flow31
Connections:
- net GND: now also J8.A1 (GND), J8.A12 (GND), J8.B1 (GND), J8.B12 (GND)
- net VBUS: now also J8.A4 (VBUS), J8.A9 (VBUS), J8.B4 (VBUS), J8.B9 (VBUS)
- net at R43.1: now also J8.A5 (CC1)
- net at U10.1 (UD+): now also J8.A6 (D-), J8.B7 (D-)
- net at U10.2 (UD-): now also J8.A7 (D+), J8.B6 (D+)
- net at R44.1: now also J8.B5 (CC2)
- net at C25.1, R41.1: now also J8.SH (SHIELD)
