File: Kicad/V2/Wrist/hand_captors.kicad_sch (KiCad schematic)
At the start: 21 parts

Commit message: j'aurai du commit avant, j'ai tunnel
Parts:
- R8: footprint (none) -> MyGlove:Resistor_0603
- renumbered C55 to C13, C56 to C14, C57 to C15, C58 to C16, C59 to C17, C60 to C18, C61 to C19, C62 to C20, C64 to C21, C63 to C22, R46 to R10, R47 to R11, R48 to R12, R49 to R13, R50 to R14, R51 to R15, R52 to R16, R54 to R17, R53 to R18, R45 to R9
