File: Kicad/V2/Wrist/captors.kicad_sch (KiCad schematic)
At the start: 7 parts, among them U3 TXS0104E

Commit message: j'aurai du commit avant, j'ai tunnel
Parts:
- removed C53, C54: 100nF, symbol G-Love:C
- removed J6: (no value), symbol G-Love:FPC_4_fingers
- removed R43, R44: 2.2K, symbol G-Love:R
- removed U3: TXS0104E, MyGlove:TXS0104EPWR, symbol G-Love:TXS0104E
- added C11, C12, C23: 100nF, MyGlove:Capacitor_0603, symbol G-Love:C
- added D1: (no value), MyGlove:TVS_DIODE, symbol G-Love:TVS_ARRAY
- added J3: (no value), MyGlove:FPC_CONNECTOR_24, symbol G-Love:FPC_CONNECTOR
- CD1: footprint MyGlove:CD4097B -> MyGlove:CD4097BPW
Connections:
- net +3.3V: now also C11.1, J3.8 (3.3V)
- net GND: now also C11.2, C12.2, C23.2, D1.3, J3.11 (GND), J3.18 (GND), J3.24 (GND), J3.3 (GNDL), J3.4 (GNDL), J3.7 (GND)
- net LED_MOSI: now also J3.5 (MOSI)
- net LED_SCK: now also J3.6 (SCK)
- net VCC: now also C12.1, C23.1
- net hand_captors/FLEX_INDEX_IN: now also J3.16 (FLEX_INDEX)
- net hand_captors/FLEX_LITTLE_IN: now also J3.23 (FLEX_LITTLE)
- net hand_captors/FLEX_MIDDLE_IN: now also J3.19 (FLEX_MIDDLE)
- net hand_captors/FLEX_RING_IN: now also J3.21 (FLEX_RING)
- net hand_captors/FLEX_THUMB_IN: now also J3.14 (FLEX_THUMB)
- net hand_captors/FORCE_INDEX_IN: now also J3.15 (FSR_INDEX)
- net hand_captors/FORCE_LITTLE_IN: now also J3.22 (FORCE_LITTLE)
- net hand_captors/FORCE_MIDDLE_IN: now also J3.17 (FSR_MIDDLE)
- net hand_captors/FORCE_RING_IN: now also J3.20 (FORCE_RING)
- net hand_captors/FORCE_THUMB_IN: now also J3.13 (FSR_THUMB)
- net hand_captors/HALL_IN: now also J3.12 (SW_HALL)
- new net VCCL: J3.1 (VCCL), J3.2 (VCCL)
- no-connect marks 10 -> 5

Commit message: Routing ADC
Connections:
- net ADC_Mux_Inhibit is gone; now on net GND: CD1.13 (INHIBIT)
- net LED_MOSI: now also D1.2
- net LED_SCK: now also D1.1
- net hand_captors/FLEX_INDEX_OUT: now also CD1.6 (X_3); no longer CD1.8 (X_1)
- net hand_captors/FLEX_LITTLE_OUT: now also CD1.19 (Y_4); no longer CD1.5 (X_4)
- net hand_captors/FLEX_MIDDLE_OUT: now also CD1.23 (Y_0); no longer CD1.7 (X_2)
- net hand_captors/FLEX_RING_OUT: now also CD1.21 (Y_2); no longer CD1.6 (X_3)
- net hand_captors/FLEX_THUMB_OUT: now also CD1.8 (X_1); no longer CD1.9 (X_0)
- net hand_captors/FORCE_INDEX_OUT: now also CD1.7 (X_2); no longer CD1.22 (Y_1)
- net hand_captors/FORCE_LITTLE_OUT: now also CD1.20 (Y_3); no longer CD1.19 (Y_4)
- net hand_captors/FORCE_MIDDLE_OUT: now also CD1.5 (X_4); no longer CD1.21 (Y_2)
- net hand_captors/FORCE_RING_OUT: now also CD1.22 (Y_1); no longer CD1.20 (Y_3)
- net hand_captors/FORCE_THUMB_OUT: now also CD1.9 (X_0); no longer CD1.23 (Y_0)
- net at J3.10 (SCL): now also D1.5
- net at J3.9 (SDA): now also D1.4
- net hand_captors/HALL_OUT: no longer names the net of CD1.18 (Y_5)
- no-connect marks 5 -> 6
