File: Kicad/V2/Wrist/touchscreen.kicad_sch (KiCad schematic)
At the start: 1 part

Commit message: j'aurai du commit avant, j'ai tunnel
Parts:
- removed J3: (no value), MyGlove:PinHeader_1x11_P2.54mm_Vertical, symbol G-Love:Conn_11_pins
- added TP2, TP3, TP4: (no value), symbol G-Love:TestPoint
Connections:
- net GND: now also TP3.1
- net VCC: now also TP2.1
- new net +3.3V: TP4.1
Other:
- note removed: "1.28 inch GC9A01 Round TFT Display"

Commit message: DRC en cours
Changed lines of the file:
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@@
-	(wire
-		(pts
-			(xy 118.11 95.25) (xy 157.48 95.25)
-		)
-		(stroke
-			(width 0)
-			(type default)
-		)
-	)
 	(wire
 		(pts
@@
 	(wire
 		(pts
-			(xy 107.95 100.33) (xy 157.48 100.33)
-		)
-		(stroke
-			(width 0)
-			(type default)
-		)
-	)
-	(wire
-		(pts
-			(xy 107.95 102.87) (xy 157.48 102.87)
-		)
-		(stroke
-			(width 0)
-			(type default)
-		)
-	)
-	(wire
-		(pts
-			(xy 107.95 97.79) (xy 118.11 97.79)
-		)
-		(stroke
-			(width 0)
-			(type default)
-		)
-	)
-	(wire
-		(pts
 			(xy 148.59 111.76) (xy 138.43 111.76)
 		)
@@
 	(wire
 		(pts
-			(xy 114.3 90.17) (xy 114.3 92.71)
-		)
-		(stroke
-			(width 0)
-			(type default)
-		)
-	)
-	(wire
-		(pts
-			(xy 107.95 105.41) (xy 157.48 105.41)
-		)
-		(stroke
-			(width 0)
-			(type default)
-		)
-	)
-	(wire
-		(pts
-			(xy 113.03 87.63) (xy 157.48 87.63)
+			(xy 124.46 97.79) (xy 107.95 97.79)
 		)
 		(stroke
@@
 	(wire
 		(pts
-			(xy 107.95 85.09) (xy 107.95 87.63)
+			(xy 124.46 107.95) (xy 107.95 107.95)
+		)
+		(stroke
+			(width 0)
+			(type default)
+		)
+	)
+	(wire
+		(pts
+			(xy 107.95 102.87) (xy 124.46 102.87)
 		)
 		(stroke
@@
 	(wire
 		(pts
-			(xy 107.95 95.25) (xy 115.57 95.25)
-		)
-		(stroke
-			(width 0)
-			(type default)
-		)
-	)
-	(wire
-		(pts
 			(xy 138.43 114.3) (xy 160.02 114.3)
 		)
@@
 	(wire
 		(pts
-			(xy 114.3 92.71) (xy 107.95 92.71)
-		)
-		(stroke
-			(width 0)
-			(type default)
-		)
-	)
-	(wire
-		(pts
-			(xy 118.11 97.79) (xy 118.11 95.25)
-		)
-		(stroke
-			(width 0)
-			(type default)
-		)
-	)
-	(wire
-		(pts
-			(xy 107.95 90.17) (xy 113.03 90.17)
+			(xy 124.46 100.33) (xy 107.95 100.33)
+		)
+		(stroke
+			(width 0)
+			(type default)
+		)
+	)
+	(wire
+		(pts
+			(xy 124.46 105.41) (xy 107.95 105.41)
 		)
 		(stroke
@@
 	(wire
 		(pts
-			(xy 107.95 85.09) (xy 157.48 85.09)
-		)
-		(stroke
-			(width 0)
-			(type default)
-		)
-	)
-	(wire
-		(pts
-			(xy 114.3 90.17) (xy 157.48 90.17)
-		)
-		(stroke
-			(width 0)
-			(type default)
-		)
-	)
-	(wire
-		(pts
-			(xy 115.57 95.25) (xy 115.57 92.71)
-		)
-		(stroke
-			(width 0)
-			(type default)
-		)
-	)
-	(wire
-		(pts
-			(xy 107.95 107.95) (xy 157.48 107.95)
-		)
-		(stroke
-			(width 0)
-			(type default)
-		)
-	)
-	(wire
-		(pts
-			(xy 115.57 92.71) (xy 157.48 92.71)
-		)
-		(stroke
-			(width 0)
-			(type default)
-		)
-	)
-	(wire
-		(pts
-			(xy 113.03 90.17) (xy 113.03 87.63)
+			(xy 107.95 92.71) (xy 124.46 92.71)
+		)
+		(stroke
+			(width 0)
+			(type default)
+		)
+	)
+	(wire
+		(pts
+			(xy 107.95 95.25) (xy 124.46 95.25)
+		)
+		(stroke
+			(width 0)
+			(type default)
+		)
+	)
+	(wire
+		(pts
+			(xy 124.46 87.63) (xy 107.95 87.63)
+		)
+		(stroke
+			(width 0)
+			(type default)
+		)
+	)
+	(wire
+		(pts
+			(xy 107.95 90.17) (xy 124.46 90.17)
 		)
 		(stroke
@@
 	(hierarchical_label "Screen_SPI_SS"
 		(shape input)
-		(at 157.48 95.25 0)
+		(at 124.46 97.79 0)
 		(effects
 			(font
@@
 	(hierarchical_label "Screen_SPI_SCK"
 		(shape input)
-		(at 157.48 85.09 0)
+		(at 124.46 102.87 0)
 		(effects
 			(font
@@
 	(hierarchical_label "Screen_SPI_MOSI"
 		(shape input)
-		(at 157.48 87.63 0)
+		(at 124.46 100.33 0)
 		(effects
 			(font
@@
 	(hierarchical_label "Touch_I2C_SDA"
 		(shape input)
-		(at 157.48 102.87 0)
+		(at 124.46 105.41 0)
 		(effects
 			(font
@@
 	(hierarchical_label "Touch_I2C_SCL"
 		(shape input)
-		(at 157.48 100.33 0)
+		(at 124.46 107.95 0)
 		(effects
 			(font
@@
 	(hierarchical_label "Screen_D{slash}C"
 		(shape input)
-		(at 157.48 92.71 0)
+		(at 124.46 95.25 0)
 		(effects
 			(font
@@
 	(hierarchical_label "Touch_I2C_INT"
 		(shape input)
-		(at 157.48 107.95 0)
+		(at 124.46 90.17 0)
 		(effects
 			(font
@@
 	(hierarchical_label "Screen_RESET"
 		(shape input)
-		(at 157.48 90.17 0)
+		(at 124.46 92.71 0)
 		(effects
 			(font
@@
 	(hierarchical_label "Touch_RESET"
 		(shape input)
-		(at 157.48 105.41 0)
-		(effects
-			(font
+		(at 124.46 87.63 0)
+		(effects
+			(font
