File: Kicad/V2/PowerArm/power.kicad_sch (KiCad schematic)
At the start: 12 parts, among them U3 AMS1117

Commit message: add routing blocks
Parts:
- J5: renamed from J_1; value Conn_USB_Receptacle -> USB Connector to Powerbank
Changed lines of the file:
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@@
 		(in_pos_files yes)
 		(dnp no)
-		(fields_autoplaced yes)
-		(property "Reference" "J_1"
+		(property "Reference" "J5"
 			(at 100.33 112.3949 0)
 			(show_name no)
@@
 			)
 		)
-		(property "Value" "Conn_USB_Receptacle"
-			(at 100.33 114.9349 0)
+		(property "Value" "USB Connector to Powerbank"
+			(at 139.192 135.636 0)
 			(show_name no)
 			(do_not_autoplace no)
@@
 			(project "PowerArm"
 				(path "/ee7054af-c2c9-421b-971c-84178cc0b718/bae02479-a44b-49ad-9522-9457ef0e9352"
-					(reference "J_1")
+					(reference "J5")
 					(unit 1)
 				)

Commit message: route power block
Parts:
- J5: footprint MyGlove:USB_C_Receptacle_GCT_USB4105-xx-A_16P_TopMnt_Horizontal -> MyGlove:USB_Conn
Changed lines of the file:
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@@
 			)
 		)
-		(property "Footprint" "MyGlove:USB_C_Receptacle_GCT_USB4105-xx-A_16P_TopMnt_Horizontal"
+		(property "Footprint" "MyGlove:USB_Conn"
 			(at 111.76 114.3 0)
 			(hide yes)

Commit message: route UART
Parts:
- removed C12, C14: 100nF, MyGlove:Capacitor_0603, symbol G-Love:C
- removed C13: 10uF, MyGlove:Capacitor_0603, symbol G-Love:C
- removed U3: AMS1117, MyGlove:AMS1117, symbol G-Love:LDO
Other:
- note removed: "LDO Sortie 3.3V"

Commit message: missing FPC addition
Parts:
- J5: footprint MyGlove:USB_Conn -> MyGlove:USB_C_Receptacle_GCT_USB4105-xx-A_16P_TopMnt_Horizontal
Changed lines of the file:
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@@
 	(text "Noise reduction"
 		(exclude_from_sim no)
-		(at 96.012 146.558 90)
+		(at 96.012 142.494 90)
 		(effects
 			(font
@@
 			)
 		)
-		(property "Footprint" "MyGlove:USB_Conn"
+		(property "Footprint" "MyGlove:USB_C_Receptacle_GCT_USB4105-xx-A_16P_TopMnt_Horizontal"
 			(at 111.76 114.3 0)
 			(hide yes)
